File: PedalBoard.kicad_pcb (KiCad board)
At the start: 2 copper layers, 26.8 x 22.4 mm, 4 parts, among them J1 Conn_01x06_Male

Commit message: layout board
Parts:
- added D2: LED, LED_THT:LED_D3.0mm, F.Cu at (75.2, 82.3)
- added D3: LED, LED_THT:LED_D3.0mm, F.Cu at (125.9, 82.3)
- added D4: LED, LED_THT:LED_D3.0mm, F.Cu at (176.8, 82.3)
- added D5: LED, LED_THT:LED_D3.0mm, F.Cu at (227.6, 82.3)
- added D6: LED, LED_THT:LED_D3.0mm, F.Cu at (278.5, 82.3)
- added R2: 1k, Resistor_THT:R_Axial_DIN0204_L3.6mm_D1.6mm_P5.08mm_Horizontal, F.Cu at (84.1, 82.3)
- added R3: 1k, Resistor_THT:R_Axial_DIN0204_L3.6mm_D1.6mm_P5.08mm_Horizontal, F.Cu at (133.6, 82.3)
- added R4: 1k, Resistor_THT:R_Axial_DIN0204_L3.6mm_D1.6mm_P5.08mm_Horizontal, F.Cu at (183.4, 82.5)
- added R5: 1k, Resistor_THT:R_Axial_DIN0204_L3.6mm_D1.6mm_P5.08mm_Horizontal, F.Cu at (236.2, 82.3)
- added R6: 1k, Resistor_THT:R_Axial_DIN0204_L3.6mm_D1.6mm_P5.08mm_Horizontal, F.Cu at (286.9, 82.3)
- added S2: SF17020F-0302-21R-L-015, SF17020F-0302-21R-L-015:SF17020F030221RL015, F.Cu at (75.2, 97.5)
- added S3: SF17020F-0302-21R-L-015, SF17020F-0302-21R-L-015:SF17020F030221RL015, F.Cu at (126.0, 97.5)
- added S4: SF17020F-0302-21R-L-015, SF17020F-0302-21R-L-015:SF17020F030221RL015, F.Cu at (176.8, 97.5)
- added S5: SF17020F-0302-21R-L-015, SF17020F-0302-21R-L-015:SF17020F030221RL015, F.Cu at (227.6, 97.5)
- added S6: SF17020F-0302-21R-L-015, SF17020F-0302-21R-L-015:SF17020F030221RL015, F.Cu at (278.4, 97.5)
- D1: value - LED + -> LED; footprint LEDs:LED_Rectangular_W3.0mm_H2.0mm -> LED_THT:LED_D3.0mm
- J1: value Conn_01x06_Male -> 8P8C; footprint Connector_PinHeader_2.00mm:PinHeader_1x06_P2.00mm_Vertical -> Connector_RJ:RJ45_Amphenol_54602-x08_Horizontal
- moved J1 75.0 mm to (155.8, 79.5), turned to 180 degrees
- moved S1 73.6 mm to (24.4, 97.5)
- moved D1 60.0 mm to (24.4, 82.3), turned to 90 degrees
- moved R1 60.0 mm to (34.5, 82.3), turned to 90 degrees
Connections:
- J1 pad 1: GND -> +9V
- J1 pad 3: Ouput -> Net-(J1-Pad3)
- J1 pad 4: FromEffect -> Net-(J1-Pad4)
- J1 pad 5: Input -> Net-(J1-Pad5)
- J1 pad 6: ToEffect -> Net-(J1-Pad6)
- R1 pad 1: Net-(J1-Pad2) -> +9V
- S1 pad 1: ToEffect -> Net-(S1-Pad1)
- S1 pad 2: Input -> Net-(J1-Pad2)
- S1 pad 3: Net-(S1-Pad3) -> GND
- S1 pad 4: FromEffect -> Net-(S1-Pad4)
- S1 pad 5: Ouput -> Net-(S1-Pad5)
- S1 pad 6: Net-(S1-Pad3) -> Net-(S1-Pad6)
- S1 pad 9: (no net) -> Net-(S1-Pad9)
Routing:
- net Net-(J1-Pad2): track 6.79 -> 149.7 mm
- net Net-(J1-Pad6): track 0.00 -> 140.6 mm
- net Net-(J1-Pad5): track 0.00 -> 130.0 mm
- net Net-(J1-Pad3): track 0.00 -> 83.1 mm
- net Net-(J1-Pad7): track 0.00 -> 51.2 mm
- net Net-(J1-Pad4): track 0.00 -> 34.7 mm
- net Net-(D5-Pad1): track 0.00 -> 23.2 mm
- net Net-(D4-Pad1): track 0.00 -> 23.2 mm
- net Net-(D6-Pad1): track 0.00 -> 22.3 mm
- net Net-(D2-Pad1): track 0.00 -> 22.2 mm
- net Net-(D3-Pad1): track 0.00 -> 22.2 mm
- net Ouput: track 19.4 -> 0.00 mm
- net FromEffect: track 18.3 -> 0.00 mm
- net ToEffect: track 17.7 -> 0.00 mm
- net Input: track 13.5 -> 0.00 mm
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- removed copper zone on B.Cu, net GND
Other:
- board size 26.8 x 22.4 mm -> 276.9 x 44.2 mm
- board text removed: "FrmE"
- board text removed: "In"
- board text removed: "LED"
- board text removed: "Out"
- board text removed: "ToEff"

Commit message: add regulator
Parts:
- added C1: 100nf, Capacitor_THT:C_Disc_D8.0mm_W2.5mm_P5.00mm, F.Cu at (219.7, 67.3)
- added C2: 10uf, Capacitor_THT:C_Disc_D8.0mm_W2.5mm_P5.00mm, F.Cu at (236.1, 67.3)
- added U1: LD1117S50TR_SOT223, Package_TO_SOT_THT:TO-220F-3_Horizontal_TabDown, F.Cu at (211.6, 76.3)
- moved R2 10.3 mm to (83.8, 72.0), turned to 270 degrees
- moved R4 10.2 mm to (183.3, 72.4), turned to 270 degrees
- moved R1 10.2 mm to (34.5, 72.1), turned to 270 degrees
- moved R3 10.2 mm to (133.6, 72.1), turned to 270 degrees
- moved R5 10.2 mm to (236.2, 72.1), turned to 270 degrees
- moved R6 10.2 mm to (286.9, 72.1), turned to 270 degrees
Connections:
- R1 pad 1: +9V -> REG_5v
- R2 pad 1: +9V -> REG_5v
- R3 pad 1: +9V -> REG_5v
- R4 pad 1: +9V -> REG_5v
- R5 pad 1: +9V -> REG_5v
- R6 pad 1: +9V -> REG_5v
Routing:
- net +9V: track 0.00 -> 72.2 mm
- added copper zone on B.Cu, net GND
- added copper zone on F.Cu, net REG_5v

Commit message: Update footswitch library
Parts:
- D1, D2, D3, D4, D5, D6: value LED -> - LED +
- S1, S2, S3, S4, S5, S6: footprint SF17020F-0302-21R-L-015:SF17020F030221RL015 -> Footswitch:Footswitch_3PDT
- moved R1 20.8 mm to (17.8, 84.5), turned to 90 degrees
- moved R2 20.2 mm to (67.9, 84.5), turned to 90 degrees
- moved R5 20.1 mm to (220.3, 84.5), turned to 90 degrees
- moved R6 19.5 mm to (271.8, 84.5), turned to 90 degrees
- moved R3 19.3 mm to (118.7, 84.5), turned to 90 degrees
- moved R4 17.8 mm to (170.2, 84.5), turned to 90 degrees
- moved C1 3.94 mm to (219.7, 71.2)
- moved C2 3.94 mm to (236.1, 71.2)
Connections:
- S1 pad 1: Net-(S1-Pad1) -> (no net)
- S1 pad 4: Net-(S1-Pad4) -> (no net)
- S1 pad 5: Net-(S1-Pad5) -> (no net)
- S1 pad 6: Net-(S1-Pad6) -> (no net)
- S1 pad 9: Net-(S1-Pad9) -> (no net)
- S2 pad 1: Net-(S2-Pad1) -> (no net)
- S2 pad 4: Net-(S2-Pad4) -> (no net)
- S2 pad 5: Net-(S2-Pad5) -> (no net)
- S2 pad 6: Net-(S2-Pad6) -> (no net)
- S2 pad 9: Net-(S2-Pad9) -> (no net)
- S3 pad 1: Net-(S3-Pad1) -> (no net)
- S3 pad 4: Net-(S3-Pad4) -> (no net)
- S3 pad 5: Net-(S3-Pad5) -> (no net)
- S3 pad 6: Net-(S3-Pad6) -> (no net)
- S3 pad 9: Net-(S3-Pad9) -> (no net)
- S4 pad 1: Net-(S4-Pad1) -> (no net)
- S4 pad 4: Net-(S4-Pad4) -> (no net)
- S4 pad 5: Net-(S4-Pad5) -> (no net)
- S4 pad 6: Net-(S4-Pad6) -> (no net)
- S4 pad 9: Net-(S4-Pad9) -> (no net)
- S5 pad 1: Net-(S5-Pad1) -> (no net)
- S5 pad 4: Net-(S5-Pad4) -> (no net)
- S5 pad 5: Net-(S5-Pad5) -> (no net)
- S5 pad 6: Net-(S5-Pad6) -> (no net)
- S5 pad 9: Net-(S5-Pad9) -> (no net)
- S6 pad 1: Net-(S6-Pad1) -> (no net)
- S6 pad 4: Net-(S6-Pad4) -> (no net)
- S6 pad 5: Net-(S6-Pad5) -> (no net)
- S6 pad 6: Net-(S6-Pad6) -> (no net)
- S6 pad 9: Net-(S6-Pad9) -> (no net)
Routing:
- net Net-(J1-Pad5): track 130.0 -> 120.0 mm
- net Net-(C1-Pad2): track 0.00 -> 6.43 mm
- net Net-(J1-Pad4): track 34.7 -> 29.2 mm
- net Net-(J1-Pad2): track 149.7 -> 144.6 mm
- net Net-(D1-Pad2): track 11.2 -> 6.76 mm
- net Net-(D2-Pad2): track 9.94 -> 7.40 mm
- net Net-(D6-Pad2): track 9.43 -> 6.89 mm
- net Net-(D5-Pad2): track 9.69 -> 7.40 mm
- net +9V: track 72.2 -> 70.6 mm
- net Net-(D3-Pad2): track 8.80 -> 7.27 mm
- net Net-(J1-Pad7): track 51.2 -> 50.2 mm
- net Net-(D4-Pad2): track 7.55 -> 6.76 mm
